Commit message: remove dae file

File: urdf/15-limo.urdf.xacro (robot description, xacro)
@@ -8,5 +8,5 @@
     <xacro:property name="base_clearance" value="-0.0" />
     <xacro:property name="M_PI" value="3.1415926536"/>
-    <xacro:macro name="limo_base" params="object_name:='limo_base' frame_link='base_link' parent_link:='base_footprint' xyz:='0 0 0' rpy:='0 0 0' color:='false' simple:='true'">
+    <xacro:macro name="limo_base" params="object_name:='limo_base' frame_link='base_link' parent_link:='base_footprint' xyz:='0 0 0' rpy:='0 0 0'">
         <xacro:property
             name="mass"
@@ -46,14 +46,7 @@
                     rpy="0 0 1.57"/>
                 <geometry>
-                    <xacro:if value="${color}">
-                        <mesh
-                            filename="file://$(find urdf_sim_tutorial)/meshes/limo_base.dae"
-                            scale="1 1 1"/>
-                    </xacro:if>
-                    <xacro:unless value="${color}">
-                        <mesh
-                            filename="file://$(find urdf_sim_tutorial)/meshes/limo_base.stl"
-                            scale="0.001 0.001 0.001"/>
-                    </xacro:unless>
+                    <mesh
+                        filename="file://$(find urdf_sim_tutorial)/meshes/limo_base.stl"
+                        scale="0.001 0.001 0.001"/>
                 </geometry>
                 <material
@@ -67,30 +60,12 @@
             <collision
                 name="${object_name}_collision">
-                <xacro:if value="${simple}">
-                    <origin
-                        xyz="0 0 ${base_height/2 - 0.025}"
-                        rpy="0 0 0"/>
-                    <geometry>
-                        <box
-                            size="${base_length} ${base_width} ${base_height}"/>
-                    </geometry>
-                </xacro:if>
-                <xacro:unless value="${simple}">
-                    <origin
-                        xyz="-0.0014 0 -0.05"
-                        rpy="0 0 1.57"/>
-                    <geometry>
-                        <xacro:if value="${color}">
-                            <mesh
-                                filename="file://$(find urdf_sim_tutorial)/meshes/limo_base.dae"
-                                scale="1 1 1"/>
-                        </xacro:if>
-                        <xacro:unless value="${color}">
-                            <mesh
-                                filename="file://$(find urdf_sim_tutorial)/meshes/limo_base.stl"
-                                scale="0.001 0.001 0.001"/>
-                        </xacro:unless>
-                    </geometry>
-                </xacro:unless>
+                <origin
+                    xyz="-0.0014 0 -0.05"
+                    rpy="0 0 1.57"/>
+                <geometry>
+                    <mesh
+                        filename="file://$(find urdf_sim_tutorial)/meshes/limo_base.stl"
+                        scale="0.001 0.001 0.001"/>
+                </geometry>
             </collision>
         </link>
@@ -116,5 +91,5 @@
         </gazebo>
     </xacro:macro>
-    <xacro:macro name="limo_wheel" params="object_name:='limo_wheel' joint_name='limo_wheel_joint' frame_link='limo_wheel_link' parent_link:='base_link' xyz:='0 0 0' rpy:='0 0 0' direction:='1' color:='false' simple:='true'">
+    <xacro:macro name="limo_wheel" params="object_name:='limo_wheel' joint_name='limo_wheel_joint' frame_link='limo_wheel_link' parent_link:='base_link' xyz:='0 0 0' rpy:='0 0 0' direction:='1'">
         <xacro:property
             name="mass"
@@ -150,14 +125,7 @@
                     rpy="0 0 0"/>
                 <geometry>
-                    <xacro:if value="${color}">
-                        <mesh
-                            filename="file://$(find urdf_sim_tutorial)/meshes/limo_wheel.dae"
-                            scale="1 1 1"/>
-                    </xacro:if>
-                    <xacro:unless value="${color}">
-                        <mesh
-                            filename="file://$(find urdf_sim_tutorial)/meshes/limo_wheel.stl"
-                            scale="0.001 0.001 0.001"/>
-                    </xacro:unless>
+                    <mesh
+                        filename="file://$(find urdf_sim_tutorial)/meshes/limo_wheel.stl"
+                        scale="0.001 0.001 0.001"/>
                 </geometry>
                 <material
@@ -170,31 +138,12 @@
             </visual>
             <collision>
-                <xacro:if value="${simple}">
-                    <origin
-                        xyz="0 0 0"
-                        rpy="${M_PI/2} 0 0"/>
-                    <geometry>
-                        <cylinder
-                            radius="${wheel_radius}"
-                            length="0.001"/>
-                    </geometry>
-                </xacro:if>
-                <xacro:unless value="${simple}">
                     <origin
                         xyz="0 ${-wheel_height/2 + 0.001} 0"
                         rpy="0 0 0"/>
                     <geometry>
-                        <xacro:if value="${color}">
-                            <mesh
-                                filename="file://$(find urdf_sim_tutorial)/meshes/limo_wheel.dae"
-                                scale="1 1 1"/>
-                        </xacro:if>
-                        <xacro:unless value="${color}">
-                            <mesh
-                                filename="file://$(find urdf_sim_tutorial)/meshes/limo_wheel.stl"
-                                scale="0.001 0.001 0.001"/>
-                        </xacro:unless>
+                        <mesh
+                            filename="file://$(find urdf_sim_tutorial)/meshes/limo_wheel.stl"
+                            scale="0.001 0.001 0.001"/>
                     </geometry>
-                </xacro:unless>
             </collision>
         </link>
@@ -610,7 +559,5 @@
         parent_link="base_footprint"
         xyz="0 0 ${wheel_radius}"
-        rpy="0 0 0"
-        simple="false"
-        color="false"/>
+        rpy="0 0 0"/>
     <xacro:limo_wheel
         object_name="wheel_front_left"
@@ -620,6 +567,5 @@
         xyz="${wheel_base/2} ${wheel_track/2} ${base_clearance}"
         rpy="0 0 0"
-        direction="1"
-        color="false"/>
+        direction="1"/>
     <xacro:limo_wheel
         object_name="wheel_front_right"
@@ -629,6 +575,5 @@
         xyz="${wheel_base/2} ${-wheel_track/2} ${base_clearance}"
         rpy="0 0 0"
-        direction="1"
-        color="false"/>
+        direction="1"/>
     <xacro:limo_wheel
         object_name="wheel_rear_left"
@@ -638,6 +583,5 @@
         xyz="${-wheel_base/2} ${wheel_track/2} ${base_clearance}"
         rpy="0 0 0"
-        direction="1"
-        color="false"/>
+        direction="1"/>
     <xacro:limo_wheel
         object_name="wheel_rear_right"
@@ -647,6 +591,5 @@
         xyz="${-wheel_base/2} ${-wheel_track/2} ${base_clearance}"
         rpy="0 0 0"
-        direction="1"
-        color="false"/>
+        direction="1"/>
     <xacro:imu
         object_name="imu"

Commit message: update urdf 15.limo

File: urdf/15-limo.urdf.xacro (robot description, xacro)
@@ -108,5 +108,5 @@
             <inertial>
                 <origin
-                    xyz="0 0 0"
+                    xyz="0 ${-wheel_height/2 + 0.001} 0"
                     rpy="0 0 0"/>
                 <mass
@@ -138,12 +138,12 @@
             </visual>
             <collision>
-                    <origin
-                        xyz="0 ${-wheel_height/2 + 0.001} 0"
-                        rpy="0 0 0"/>
-                    <geometry>
-                        <mesh
-                            filename="file://$(find urdf_sim_tutorial)/meshes/limo_wheel.stl"
-                            scale="0.001 0.001 0.001"/>
-                    </geometry>
+                <origin
+                    xyz="0 ${-wheel_height/2 + 0.001} 0"
+                    rpy="0 0 0"/>
+                <geometry>
+                    <mesh
+                        filename="file://$(find urdf_sim_tutorial)/meshes/limo_wheel.stl"
+                        scale="0.001 0.001 0.001"/>
+                </geometry>
             </collision>
         </link>
@@ -512,5 +512,4 @@
                 <state_interface name="position"/>
                 <state_interface name="velocity"/>
-                <command_interface name="position"/>
                 <command_interface name="velocity">
                     <param name="min">-10</param>
@@ -521,5 +520,4 @@
                 <state_interface name="position"/>
                 <state_interface name="velocity"/>
-                <command_interface name="position"/>
                 <command_interface name="velocity">
                     <param name="min">-10</param>
@@ -530,5 +528,4 @@
                 <state_interface name="position"/>
                 <state_interface name="velocity"/>
-                <command_interface name="position"/>
                 <command_interface name="velocity">
                     <param name="min">-10</param>
@@ -539,5 +536,4 @@
                 <state_interface name="position"/>
                 <state_interface name="velocity"/>
-                <command_interface name="position"/>
                 <command_interface name="velocity">
                     <param name="min">-10</param>
@@ -574,6 +570,6 @@
         parent_link="base_link"
         xyz="${wheel_base/2} ${-wheel_track/2} ${base_clearance}"
-        rpy="0 0 0"
-        direction="1"/>
+        rpy="0 0 ${M_PI}"
+        direction="-1"/>
     <xacro:limo_wheel
         object_name="wheel_rear_left"
@@ -590,6 +586,6 @@
         parent_link="base_link"
         xyz="${-wheel_base/2} ${-wheel_track/2} ${base_clearance}"
-        rpy="0 0 0"
-        direction="1"/>
+        rpy="0 0 ${M_PI}"
+        direction="-1"/>
     <xacro:imu
         object_name="imu"
